File: pcb/mini_2.0/breezedude_mini.kicad_pcb (KiCad board)
At the start: 2 copper layers, 53 x 22.5 mm, 49 parts, among them J1 Conn_01x02_Pin, J2 Conn_01x04_Pin, J3 Conn_01x04_Pin, J4 Conn_01x03_Pin, J5 Conn_01x04_Pin, J6 Conn_01x02_Pin, J7 USB_C_Receptacle_USB2.0_16P, J8 Conn_01x02_Pin, Q1 P-MOS, Q2 P-MOS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

Commit message: V2.3: * Added 10k pullup to Ssensor UART RX to aboid wakeup when no sensor is connected/cable failiure * Replaced CN3063 with TP4057 for better avaliability. * Moved SWD connector for better acessibility * RF optimisation
Parts:
- removed U1: PMIC-CN3063_SOIC8_, Package_SO:Infineon_PG-DSO-8-43
- added R12: 10k, Resistor_SMD:R_0402_1005Metric, F.Cu at (119.9, 107.5)
- added U9: TP4057, Package_TO_SOT_SMD:TSOT-23-6, F.Cu at (142.2, 119.8)
- moved U7 17.8 mm to (91.2, 112.8), turned to -90 degrees
- moved U5 17.5 mm to (92.8, 116.1), turned to 90 degrees
- moved C11 12.4 mm to (139.9, 122.6)
- moved U4 11.0 mm to (89.0, 116.3), turned to 180 degrees
- moved C10 10.6 mm to (89.1, 118.7), turned to 180 degrees
- moved C1 6.63 mm to (142.6, 122.6), turned to 0 degrees
- moved JP1 5.16 mm to (147.4, 119.2)
- moved R1 4.94 mm to (145.0, 119.4), turned to -90 degrees
- moved C2 0.99 mm to (135.2, 111.7), turned to 180 degrees
- moved J4 0.92 mm to (135.3, 108.4)
- moved J1 0.29 mm to (145.8, 109.8)
Routing:
- net /SOLAR+: track 18.7 -> 25.8 mm
- net VCC_WS: track 19.1 -> 25.3 mm, vias 1 -> 2
- net Net-(JP1-A): track 28.4 -> 23.3 mm
- net GND: track 23.1 -> 18.2 mm, vias 53 -> 62
- net /BATT+: track 34.6 -> 30.5 mm
- net /PV_CHARGE: track 15.4 -> 11.7 mm
- net /PV_DONE: track 13.8 -> 16.1 mm
- net /RESET: track 16.9 -> 18.9 mm
- net Net-(U9-PROG): track 3.73 -> 1.77 mm
- net Net-(D5-A): track 2.80 -> 4.38 mm
- net /RX: track 8.50 -> 9.70 mm
- net /SDA: track 52.9 -> 52.1 mm
- net /SCL: track 55.2 -> 54.5 mm
- net /SWDCLK: track 2.17 -> 2.86 mm
- net SW_WS: track 5.19 -> 4.51 mm
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Other:
- board text added: "ANT"
- board text added: "V2.3"
- board text removed: "V2.2"
