File: pcb/mini_2.0/breezedude_mini.kicad_sch (KiCad schematic)
At the start: 49 parts, among them J1 Conn_01x02_Pin, J2 Conn_01x04_Pin, J3 Conn_01x04_Pin, J4 Conn_01x03_Pin, J5 Conn_01x04_Pin, J6 Conn_01x02_Pin, J7 USB_C_Receptacle_USB2.0_16P, J8 Conn_01x02_Pin, Q1 P-MOS, Q2 P-MOS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

Commit message: V2.3: * Added 10k pullup to Ssensor UART RX to aboid wakeup when no sensor is connected/cable failiure * Replaced CN3063 with TP4057 for better avaliability. * Moved SWD connector for better acessibility * RF optimisation
Parts:
- removed U1: PMIC-CN3063_SOIC8_, Package_SO:Infineon_PG-DSO-8-43, symbol PMIC-CN3063_SOIC8_:PMIC-CN3063_SOIC8_
- added R12: 10k, Resistor_SMD:R_0402_1005Metric, symbol Device:R
- added U9: TP4057, Package_TO_SOT_SMD:TSOT-23-6, symbol Battery_Management:TP4057
Connections:
- net BATT+: now also U9.3 (BAT)
- net GND: now also U9.2 (GND)
- net PV_CHARGE: now also U9.1 (~{CHRG})
- net PV_DONE: now also U9.5 (STDBY)
- net RX: now also R12.1
- net SOLAR+: now also U9.4 (V_{CC})
- net VCC_WS: now also R12.2
- net at R1.1: now also U9.6 (PROG)
Other:
- moved on the sheet: R1
